Commit message: Modify xacro

File: description/robot_core.xacro (robot description, xacro)
@@ -38,4 +38,7 @@
         </geometry>
     </collision>
+    <xacro:inertial_box mass="0.5" x="0.3" y="0.3" z="0.15">
+       <origin xyz="0.15 0.0 0.075" rpy= "0 0 0"/>
+    </xacro:inertial_box>
  </link>
  <!--Left Wheel Link-->
@@ -59,4 +62,7 @@
         </geometry>
     </collision>
+    <xacro:inertial_cylinder mass="0.5" length="0.04" radius="0.05">
+       <origin xyz="0.0 0.0 0.0" rpy="0.0 0.0 0.0"/>
+    </xacro:inertial_cylinder>
  </link>
  <!--Right Wheel Link-->
@@ -80,4 +86,7 @@
         </geometry>
     </collision>
+    <xacro:inertial_cylinder mass="0.5" length="0.04" radius="0.05">
+       <origin xyz="0.0 0.0 0.0" rpy="0.0 0.0 0.0"/>
+    </xacro:inertial_cylinder>
  </link>
   <!--Caster Wheel Link-->
@@ -100,4 +109,7 @@
         </geometry>
     </collision>
+    <xacro:inertial_sphere mass="0.1" radius="0.05">
+     <origin xyz="0.0 0.0 0.0" rpy="0.0 0.0 0.0"/>
+    </xacro:inertial_sphere>
 </link>
 </robot>

Commit message: Add Gazebo material colors

File: description/robot_core.xacro (robot description, xacro)
@@ -42,4 +42,7 @@
     </xacro:inertial_box>
  </link>
+ <gazebo reference="chassis">
+        <material>Gazebo/White</material>
+    </gazebo>
  <!--Left Wheel Link-->
  <joint name="left_wheel_joint" type="continuous">
@@ -66,4 +69,7 @@
     </xacro:inertial_cylinder>
  </link>
+ <gazebo reference="left_wheel">
+        <material>Gazebo/Blue</material>
+    </gazebo>
  <!--Right Wheel Link-->
   <joint name="right_wheel_joint" type="continuous">
@@ -90,4 +96,7 @@
     </xacro:inertial_cylinder>
  </link>
+ <gazebo reference="right_wheel">
+        <material>Gazebo/Blue</material>
+    </gazebo>
   <!--Caster Wheel Link-->
   <joint name="caster_wheel_joint" type="fixed">
@@ -113,3 +122,6 @@
     </xacro:inertial_sphere>
 </link>
+<gazebo reference="caster_wheel">
+        <material>Gazebo/Black</material>
+    </gazebo>
 </robot>
