Commit message: modify lidar

File: description/lidar.xacro (robot description, xacro)
@@ -1,39 +1,37 @@
 <?xml version="1.0"?>
-<robot xmlns:xacro="http://www.ros.org/wiki/xacro">
-   <joint name="laser_joint" type="fixed">
+<robot xmlns:xacro="http://www.ros.org/wiki/xacro" >
+    <joint name="laser_joint" type="fixed">
         <parent link="chassis"/>
         <child link="laser_frame"/>
-        <origin xyz="0.1 0.0 0.175" rpy="0.0 0.0 0.0"/>
-   </joint>
+        <origin xyz="0.1 0 0.175" rpy="0 0 0"/>
+    </joint>
     <link name="laser_frame">
         <visual>
-        <geometry>
-            <cylinder radius="0.05" length="0.04"/>
-        </geometry>
-        <material name="red">
-        </material>
-    </visual>
-    <collision>
-        <geometry>
-            <cylinder radius="0.05" length="0.04"/>
-        </geometry>
-    </collision>
-    <xacro:inertial_cylinder mass="0.5" length="0.04" radius="0.05">
-       <origin xyz="0.0 0.0 0.0" rpy="0.0 0.0 0.0"/>
-    </xacro:inertial_cylinder>
+            <geometry>
+                <cylinder radius="0.05" length="0.04"/>
+            </geometry>
+            <material name="red"/>
+        </visual>
+        <collision>
+            <geometry>
+                <cylinder radius="0.05" length="0.04"/>
+            </geometry>
+        </collision>
+        <xacro:inertial_cylinder mass="0.1" length="0.04" radius="0.05">
+            <origin xyz="0 0 0" rpy="0 0 0"/>
+        </xacro:inertial_cylinder>
     </link>
     <gazebo reference="laser_frame">
-    <material>Gazebo/Red</material>
-        <sensor name="laser" typre="ray">
+        <material>Gazebo/Red</material>
+        <sensor name="laser" type="ray">
             <pose> 0 0 0 0 0 0 </pose>
-            <visualize> true</visualize>
-            <update_rate>true</update_rate>
+            <visualize>true</visualize>
+            <update_rate>10</update_rate>
             <ray>
                 <scan>
                     <horizontal>
                         <samples>360</samples>
-                        <resolution>1</resolution>
                         <min_angle>-3.14</min_angle>
-                        <max_angle> 3.14</max_angle>
+                        <max_angle>3.14</max_angle>
                     </horizontal>
                 </scan>
@@ -41,5 +39,4 @@
                     <min>0.3</min>
                     <max>12</max>
-                    <resolution>0.01</resolution>
                 </range>
             </ray>

File: description/robot_core.xacro (robot description, xacro)
@@ -121,5 +121,5 @@
         </geometry>
     </collision>
-    <xacro:inertial_sphere mass="0.1" radius="0.05">
+    <xacro:inertial_sphere mass="0.3" radius="0.05">
      <origin xyz="0.0 0.0 0.0" rpy="0.0 0.0 0.0"/>
     </xacro:inertial_sphere>
